Commit message: feat(wa1-description): add live RViz2 visualization
Provide static and live display launch files with bridge joint feedback mapping.

Simplify the ROS 2 description package, remove legacy assembly resources, track meshes with Git LFS, and update documentation.

File: src/wa1_description/urdf/WA1_400L.urdf (robot description, URDF)
Before this commit: robot WA1_400L, 64 links, 63 joints
Links:
- removed link HAND_L
- removed link HAND_R
- removed link index_Link1_L
- removed link index_Link1_R
- removed link index_Link2_L
- removed link index_Link2_R
- removed link index_Link3_L
- removed link index_Link3_R
- removed link little_Link1_L
- removed link little_Link1_R
- removed link little_Link2_L
- removed link little_Link2_R
- removed link little_Link3_L
- removed link little_Link3_R
- removed link middle_Link1_L
- removed link middle_Link1_R
- removed link middle_Link2_L
- removed link middle_Link2_R
- removed link middle_Link3_L
- removed link middle_Link3_R
- removed link ring_Link1_L
- removed link ring_Link1_R
- removed link ring_Link2_L
- removed link ring_Link2_R
- removed link ring_Link3_L
- removed link ring_Link3_R
- removed link thumb_Link1_L
- removed link thumb_Link1_R
- removed link thumb_Link2_L
- removed link thumb_Link2_R
- removed link thumb_Link3_L
- removed link thumb_Link3_R
Joints:
- removed joint Hand_L
- removed joint Hand_R
- removed joint index_DIP_L
- removed joint index_DIP_R
- removed joint index_MCP_L
- removed joint index_MCP_R
- removed joint index_PIP_L
- removed joint index_PIP_R
- removed joint little_DIP_L
- removed joint little_DIP_R
- removed joint little_MCP_L
- removed joint little_MCP_R
- removed joint little_PIP_L
- removed joint little_PIP_R
- removed joint middle_DIP_L
- removed joint middle_DIP_R
- removed joint middle_MCP_L
- removed joint middle_MCP_R
- removed joint middle_PIP_L
- removed joint middle_PIP_R
- removed joint ring_DIP_L
- removed joint ring_DIP_R
- removed joint ring_MCP_L
- removed joint ring_MCP_R
- removed joint ring_PIP_L
- removed joint ring_PIP_R
- removed joint thumb_CMC_L
- removed joint thumb_CMC_R
- removed joint thumb_IP_L
- removed joint thumb_IP_R
- removed joint thumb_MP_L
- removed joint thumb_MP_R

Commit message: feat(wa1_description): add camera link

File: src/wa1_description/urdf/WA1_400L.urdf (robot description, URDF)
Before this commit: robot WA1_400L, 32 links, 31 joints
Links:
- added link head_camera_d435i_link
Joints:
- added joint head_camera_d435i_joint: type fixed, parent HEAD, child head_camera_d435i_link, origin xyz=0.0651401529140153 0 0.112439207885702 rpy=0 0.261799387799031 0, axis 0 0 0
